File: TLink.kicad_sch (KiCad schematic)
At the start: 17 parts, among them J1 ZH_01x06, J2 TYPEC-304S-ACP16, P1 RT9013-33GB, SW1 SW_SPST, U1 CH549F

Commit message: TLink v1.1 For ARM/RISC-V
Connections:
- net +3V3: now also D1.1 (K), D2.1 (K), SW1.2 (B)
- net GND: no longer D1.1 (K), D2.1 (K), SW1.2 (B)
Changed lines of the file:
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@@
     )
   )
-  (symbol (lib_id "power:GND") (at 160.655 133.35 90) (unit 1)
-    (in_bom yes) (on_board yes) (dnp no) (fields_autoplaced)
-    (property "Reference" "#PWR032" (at 167.005 133.35 0)
-      (effects (font (size 1.27 1.27)) hide)
-    )
-    (property "Value" "GND" (at 164.465 133.985 90)
-      (effects (font (size 1.27 1.27)) (justify right))
+  (symbol (lib_id "power:+3V3") (at 160.655 133.35 270) (unit 1)
+    (in_bom yes) (on_board yes) (dnp no) (fields_autoplaced)
+    (property "Reference" "#PWR031" (at 156.845 133.35 0)
+      (effects (font (size 1.27 1.27)) hide)
+    )
+    (property "Value" "+3V3" (at 163.83 133.985 90)
+      (effects (font (size 1.27 1.27)) (justify left))
     )
     (property "Footprint" "" (at 160.655 133.35 0)
@@
       (project "Bomb"
         (path "/194c1727-0946-408e-8b51-f6390044346e"
-          (reference "#PWR032") (unit 1)
+          (reference "#PWR031") (unit 1)
         )
       )
@@
       (project "kicad"
         (path "/f78cadc8-bca9-496e-9ea2-5c75586d48dd"
-          (reference "#PWR016") (unit 1)
+          (reference "#PWR017") (unit 1)
         )
       )
@@
     )
   )
+  (symbol (lib_id "power:+3V3") (at 116.205 126.365 270) (unit 1)
+    (in_bom yes) (on_board yes) (dnp no) (fields_autoplaced)
+    (property "Reference" "#PWR031" (at 112.395 126.365 0)
+      (effects (font (size 1.27 1.27)) hide)
+    )
+    (property "Value" "+3V3" (at 119.38 127 90)
+      (effects (font (size 1.27 1.27)) (justify left))
+    )
+    (property "Footprint" "" (at 116.205 126.365 0)
+      (effects (font (size 1.27 1.27)) hide)
+    )
+    (property "Datasheet" "" (at 116.205 126.365 0)
+      (effects (font (size 1.27 1.27)) hide)
+    )
+    (pin "1")
+    (instances
+      (project "Bomb"
+        (path "/194c1727-0946-408e-8b51-f6390044346e"
+          (reference "#PWR031") (unit 1)
+        )
+      )
+      (project "TLink"
+        (path "/4bc051d4-ecec-4cff-9a14-729c7b84e105"
+          (reference "#PWR01") (unit 1)
+        )
+      )
+      (project "kicad"
+        (path "/f78cadc8-bca9-496e-9ea2-5c75586d48dd"
+          (reference "#PWR017") (unit 1)
+        )
+      )
+    )
+  )
+  (symbol (lib_id "power:+3V3") (at 160.655 124.46 270) (unit 1)
+    (in_bom yes) (on_board yes) (dnp no) (fields_autoplaced)
+    (property "Reference" "#PWR031" (at 156.845 124.46 0)
+      (effects (font (size 1.27 1.27)) hide)
+    )
+    (property "Value" "+3V3" (at 163.83 125.095 90)
+      (effects (font (size 1.27 1.27)) (justify left))
+    )
+    (property "Footprint" "" (at 160.655 124.46 0)
+      (effects (font (size 1.27 1.27)) hide)
+    )
+    (property "Datasheet" "" (at 160.655 124.46 0)
+      (effects (font (size 1.27 1.27)) hide)
+    )
+    (pin "1")
+    (instances
+      (project "Bomb"
+        (path "/194c1727-0946-408e-8b51-f6390044346e"
+          (reference "#PWR031") (unit 1)
+        )
+      )
+      (project "TLink"
+        (path "/4bc051d4-ecec-4cff-9a14-729c7b84e105"
+          (reference "#PWR023") (unit 1)
+        )
+      )
+      (project "kicad"
+        (path "/f78cadc8-bca9-496e-9ea2-5c75586d48dd"
+          (reference "#PWR017") (unit 1)
+        )
+      )
+    )
+  )
   (symbol (lib_id "Device:R_Small") (at 184.15 96.52 0) (unit 1)
     (in_bom yes) (on_board yes) (dnp no) (fields_autoplaced)
@@
         (path "/4bc051d4-ecec-4cff-9a14-729c7b84e105"
           (reference "#FLG02") (unit 1)
-        )
-      )
-    )
-  )
-  (symbol (lib_id "power:GND") (at 160.655 124.46 90) (unit 1)
-    (in_bom yes) (on_board yes) (dnp no) (fields_autoplaced)
-    (property "Reference" "#PWR032" (at 167.005 124.46 0)
-      (effects (font (size 1.27 1.27)) hide)
-    )
-    (property "Value" "GND" (at 164.465 125.095 90)
-      (effects (font (size 1.27 1.27)) (justify right))
-    )
-    (property "Footprint" "" (at 160.655 124.46 0)
-      (effects (font (size 1.27 1.27)) hide)
-    )
-    (property "Datasheet" "" (at 160.655 124.46 0)
-      (effects (font (size 1.27 1.27)) hide)
-    )
-    (pin "1")
-    (instances
-      (project "Bomb"
-        (path "/194c1727-0946-408e-8b51-f6390044346e"
-          (reference "#PWR032") (unit 1)
-        )
-      )
-      (project "TLink"
-        (path "/4bc051d4-ecec-4cff-9a14-729c7b84e105"
-          (reference "#PWR023") (unit 1)
-        )
-      )
-      (project "kicad"
-        (path "/f78cadc8-bca9-496e-9ea2-5c75586d48dd"
-          (reference "#PWR016") (unit 1)
         )
       )
@@
         )
       )
-    )
-  )
-  (symbol (lib_id "power:GND") (at 116.205 126.365 90) (unit 1)
-    (in_bom yes) (on_board yes) (dnp no) (fields_autoplaced)
-    (property "Reference" "#PWR094" (at 122.555 126.365 0)
-      (effects (font (size 1.27 1.27)) hide)
-    )
-    (property "Value" "GND" (at 119.38 127 90)
-      (effects (font (size 1.27 1.27)) (justify right))
-    )
-    (property "Footprint" "" (at 116.205 126.365 0)
-      (effects (font (size 1.27 1.27)) hide)
-    )
-    (property "Datasheet" "" (at 116.205 126.365 0)
-      (effects (font (size 1.27 1.27)) hide)
-    )
-    (pin "1")
-    (instances
-      (project "Bomb"
-        (path "/194c1727-0946-408e-8b51-f6390044346e"
-          (reference "#PWR094") (unit 1)
-        )
-      )
-      (project "TLink"
-        (path "/4bc051d4-ecec-4cff-9a14-729c7b84e105"
-          (reference "#PWR01") (unit 1)
-        )
-      )
